Commit message: change the color of macanum_car

File: macanum_car/ares_description/urdf/ares_base.xacro (robot description, xacro)
@@ -2,4 +2,7 @@
 <robot name="ares_base" xmlns:xacro="http://www.ros.org/wiki/xacro">
 	<xacro:macro name="ares_base">
+	  <gazebo reference="base_link">
+    	<material>Gazebo/FlatBlack</material>
+  	  </gazebo>
 		<link name="base_link">
 			<inertial>
@@ -13,7 +16,4 @@
 					<mesh filename="package://ares_description/meshes/base_link.STL" />
 				</geometry>
-				<material name="">
-					<color rgba="0.10196 0.10196 0.10196 1" />
-				</material>
 			</visual>
 			<collision>
@@ -24,4 +24,7 @@
 			</collision>
 		</link>
+	  <gazebo reference="wheel_lf_link">
+    	 <material>Gazebo/DarkGrey</material>
+  	  </gazebo>
 		<link name="wheel_lf_link">
 			<inertial>
@@ -35,7 +38,4 @@
 					<mesh filename="package://ares_description/meshes/wheel_lf_link.STL" />
 				</geometry>
-				<material name="">
-					<color rgba="0.79216 0.81961 0.93333 1" />
-				</material>
 			</visual>
 			<collision>
@@ -52,4 +52,7 @@
 			<axis xyz="0 -1 0" />
 		</joint>
+		<gazebo reference="wheel_lb_link">
+    			<material>Gazebo/DarkGrey</material>
+  	    	</gazebo>
 		<link name="wheel_lb_link">
 			<inertial>
@@ -63,7 +66,4 @@
 					<mesh filename="package://ares_description/meshes/wheel_lb_link.STL" />
 				</geometry>
-				<material name="">
-					<color rgba="0.79216 0.81961 0.93333 1" />
-				</material>
 			</visual>
 			<collision>
@@ -80,4 +80,7 @@
 			<axis xyz="0 -1 0" />
 		</joint>
+		<gazebo reference="wheel_rf_link">
+    		<material>Gazebo/DarkGrey</material>
+  	    </gazebo>
 		<link name="wheel_rf_link">
 			<inertial>
@@ -91,7 +94,4 @@
 					<mesh filename="package://ares_description/meshes/wheel_rf_link.STL" />
 				</geometry>
-				<material name="">
-					<color rgba="0.79216 0.81961 0.93333 1" />
-				</material>
 			</visual>
 			<collision>
@@ -108,4 +108,7 @@
 			<axis xyz="0 -1 0" />
 		</joint>
+		<gazebo reference="wheel_rb_link">
+    		<material>Gazebo/DarkGrey</material>
+  	    </gazebo>
 		<link name="wheel_rb_link">
 			<inertial>
@@ -119,7 +122,4 @@
 					<mesh filename="package://ares_description/meshes/wheel_rb_link.STL" />
 				</geometry>
-				<material name="">
-					<color rgba="0.79216 0.81961 0.93333 1" />
-				</material>
 			</visual>
 			<collision>
@@ -136,4 +136,7 @@
 			<axis xyz="0 -1 0" />
 		</joint>
+		<gazebo reference="controller_link">
+    		<material>Gazebo/DarkGrey</material>
+  	    </gazebo>
 		<link name="controller_link">
 			<inertial>
@@ -147,7 +150,4 @@
 					<mesh filename="package://ares_description/meshes/controller_link.STL" />
 				</geometry>
-				<material name="">
-					<color rgba="1 1 1 1" />
-				</material>
 			</visual>
 			<collision>
@@ -163,4 +163,11 @@
 			<child link="controller_link" />
 			<axis xyz="0 0 0" />
+		</joint>
+		<!--The root link base_link has an inertia specified in the URDF, but KDL does not support a root link with an inertia.  As a workaround, you can add an extra dummy link to your URDF. -->
+		<link name="dummy">
+		</link>
+		<joint name="dummy_joint" type="fixed">
+     		<parent link="dummy"/>
+     		<child link="base_link"/>
 		</joint>
 		<gazebo>

File: macanum_car/ares_description/urdf/ares_laser.xacro (robot description, xacro)
@@ -10,5 +10,5 @@
     <xacro:property name="camera_offset_x" value="0" />
     <xacro:property name="camera_offset_y" value="0" />
-    <xacro:property name="camera_offset_z" value="0.2" />
+    <xacro:property name="camera_offset_z" value="0.11" />
     <!-- Camera -->
     <joint name="camera_joint" type="fixed">

File: macanum_car/ares_description/urdf/sensors/camera.xacro (robot description, xacro)
@@ -3,4 +3,7 @@
     <xacro:macro name="camera" params="prefix:=camera">
         <!-- Create laser reference frame -->
+        <gazebo reference="${prefix}_link">
+    	    <material>Gazebo/FlatBlack</material>
+  	</gazebo>
         <link name="${prefix}_link">
             <inertial>
@@ -14,18 +17,14 @@
                 <origin xyz=" 0 0 0 " rpy="0 0 0" />
                 <geometry>
-                    <box size="0.01 0.04 0.04" />
+                    <box size="0.01 0.02 0.02" />
                 </geometry>
-                <material name="black"/>
             </visual>
             <collision>
                 <origin xyz="0.0 0.0 0.0" rpy="0 0 0" />
                 <geometry>
-                    <box size="0.01 0.04 0.04" />
+                    <box size="0.01 0.02 0.02" />
                 </geometry>
             </collision>
         </link>
-        <gazebo reference="${prefix}_link">
-            <material>Gazebo/Black</material>
-        </gazebo>
         <gazebo reference="${prefix}_link">
             <sensor type="camera" name="camera_node">

File: macanum_car/ares_description/urdf/sensors/laser.xacro (robot description, xacro)
@@ -2,4 +2,7 @@
 <robot name="laser" xmlns:xacro="http://www.ros.org/wiki/xacro">
 	<xacro:macro name="laser">
+	<gazebo reference="laser_link">
+    		<material>Gazebo/DarkGrey</material>
+  	</gazebo>
 		<link name="laser_link">
 			<inertial>
@@ -13,7 +16,4 @@
 					<mesh filename="package://ares_description/meshes/laser_link.STL" />
 				</geometry>
-				<material name="">
-					<color rgba="0.79216 0.81961 0.93333 1" />
-				</material>
 			</visual>
 			<collision>

Commit message: not important

File: macanum_car/ares_description/urdf/ares_base.xacro (robot description, xacro)
@@ -3,5 +3,5 @@
 	<xacro:macro name="ares_base">
 	  <gazebo reference="base_link">
-    	<material>Gazebo/FlatBlack</material>
+    	<material>Gazebo/BlueGlow</material>
   	  </gazebo>
 		<link name="base_link">
